Commit message: update quad urdf

File: resources/robots/Pikachu_V025/urdf/Pikachu_V025_flat_18dof.urdf (robot description, URDF)
Before this commit: robot Pikachu_V025, 19 links, 18 joints
Links:
- removed link left_elbow_link
- removed link right_elbow_link
- added link left_elbow_ankle_link, mass 0.0144258718112896; collision mesh filename=../meshes/left_elbow_link.STL; visual mesh filename=../meshes/left_elbow_link.STL
- added link right_elbow_ankle_link, mass 0.0144258718112896; collision mesh filename=../meshes/right_elbow_link.STL; visual mesh filename=../meshes/right_elbow_link.STL
Joints:
- joint left_elbow_joint: child left_elbow_link -> left_elbow_ankle_link
- joint right_elbow_joint: child right_elbow_link -> right_elbow_ankle_link

File: resources/robots/Pikachu_V025/urdf/Pikachu_V025_flat_18dof_quad.urdf (robot description, URDF)
Before this commit: robot Pikachu_V025, 20 links, 19 joints
Joints:
- joint left_ankle_joint: axis 0 -1 0 -> 0 1 0; limit lower=-0.52 upper=1.05 effort=9.0 velocity=2 -> lower=-1.05 upper=0.52   effort=9.0 velocity=2
- joint left_arm_pitch_joint: axis 0 -1 0 -> 0 1 0; limit lower=-1.05 upper=3.14 effort=9 velocity=2 -> lower=-3.14 upper=1.05 effort=9 velocity=2
- joint left_arm_yaw_joint: axis 0 0 1 -> 0 0 -1
- joint left_elbow_ankle_joint: axis 0 -1 0 -> 0 1 0; limit lower=0 upper=2.44 effort=9 velocity=2 -> lower=-2.44 upper=0 effort=9 velocity=2
- joint left_hip_pitch_joint: axis 0 -1 0 -> 0 1 0; limit lower=0 upper=2.44 effort=12.5 velocity=2 -> lower=-2.44 upper=0 effort=12.5 velocity=2
- joint left_hip_yaw_joint: axis 0 0 1 -> 0 0 -1; limit lower=-0.09 upper=0.26 effort=9.0 velocity=1 -> lower=-0.26 upper=0.09 effort=9.0 velocity=1
- joint left_knee_joint: axis 0 1 0 -> 0 -1 0; limit lower=0 upper=1.57 effort=12.5 velocity=3 -> lower=-1.57 upper=0 effort=12.5 velocity=3
- joint right_arm_roll_joint: axis -1 0 0 -> 1 0 0; limit lower=0.0 upper=1.57 effort=9 velocity=2 -> lower=-1.57 upper=0 effort=9 velocity=2
- joint right_arm_yaw_joint: axis 0 0 1 -> 0 0 -1
- joint right_hip_roll_joint: axis -1 0 0 -> 1 0 0; limit lower=-0.09 upper=0.26 effort=9.0 velocity=1 -> lower=-0.26 upper=0.09 effort=9.0 velocity=1
