Commit message: update quad config

File: resources/robots/Pikachu_V025/urdf/Pikachu_V025_flat_18dof_quad.urdf (robot description, URDF)
Before this commit: robot Pikachu_V025, 20 links, 19 joints
Joints:
- joint left_arm_yaw_joint: type revolute -> fixed
- joint left_elbow_ankle_joint: type revolute -> fixed
- joint right_arm_yaw_joint: type revolute -> fixed
- joint right_elbow_ankle_joint: type revolute -> fixed
