Commit message: add rolling

File: resources/robots/Pikachu_V025/urdf/Pikachu_V025_flat_14dof_quad.urdf (robot description, URDF)
Before this commit: robot Pikachu_V025, 23 links, 22 joints
Joints:
- joint world_to_base: origin xyz=0 0 0 rpy=0 1.5708 0 -> xyz=0 0 0 rpy=0 1.7708 0

Commit message: fix world origin

File: resources/robots/Pikachu_V025/urdf/Pikachu_V025_flat_14dof_quad.urdf (robot description, URDF)
Before this commit: robot Pikachu_V025, 23 links, 22 joints
Joints:
- joint world_to_base: origin xyz=0 0 0 rpy=0 1.7708 0 -> xyz=0 0 0 rpy=0 1.5708 0
